Commit message: modified the xacro for uid based spawns

File: src/bot_description/urdf/bot_grid.xacro (robot description, xacro)
@@ -1,104 +1,110 @@
 <?xml version="1.0" ?>
 <robot name="bot_grid" xmlns:xacro="http://www.ros.org/wiki/xacro">
-<xacro:include filename="$(find bot_description)/urdf/materials_bot.xacro" />
-<xacro:include filename="$(find bot_description)/urdf/bot_grid.trans" />
-<xacro:include filename="$(find bot_description)/urdf/bot_grid.gazebo" />
-<link name="base_link">
-  <inertial>
-    <origin rpy="0 0 0" xyz="0.0 0.0 0.027415539003148855"/>
-    <mass value="1.1517833070915058"/>
-    <inertia ixx="0.001068" ixy="-2.4e-05" ixz="-8e-06" iyy="0.000918" iyz="4.8e-05" izz="0.001472"/>
-  </inertial>
-  <visual>
-    <origin rpy="0 0 0" xyz="0 0 0"/>
-    <geometry>
-      <mesh filename="package://bot_description/meshes/base_link.stl" scale="0.001 0.001 0.001"/>
-    </geometry>
-    <material name="silver"/>
-  </visual>
-  <collision>
-    <origin rpy="0 0 0" xyz="0 0 0"/>
-    <geometry>
-      <mesh filename="package://bot_description/meshes/base_link.stl" scale="0.001 0.001 0.001"/>
-    </geometry>
-  </collision>
-</link>
-<link name="rod_1">
-  <inertial>
-    <origin rpy="0 0 0" xyz="-0.03412970107262531 3.283082382239677e-07 0.000999532672142013"/>
-    <mass value="0.004917856385932786"/>
-    <inertia ixx="0.0" ixy="0.0" ixz="-0.0" iyy="2e-06" iyz="-0.0" izz="2e-06"/>
-  </inertial>
-  <visual>
-    <origin rpy="0 0 0" xyz="-0.021523 -0.007087 -0.04083"/>
-    <geometry>
-      <mesh filename="package://bot_description/meshes/rod_1.stl" scale="0.001 0.001 0.001"/>
-    </geometry>
-    <material name="silver"/>
-  </visual>
-  <collision>
-    <origin rpy="0 0 0" xyz="-0.021523 -0.007087 -0.04083"/>
-    <geometry>
-      <mesh filename="package://bot_description/meshes/rod_1.stl" scale="0.001 0.001 0.001"/>
-    </geometry>
-  </collision>
-</link>
-<link name="wheel_right_1">
-  <inertial>
-    <origin rpy="0 0 0" xyz="-0.0033351165545466577 4.777016239451704e-07 -1.512305142191417e-07"/>
-    <mass value="0.03301117951310708"/>
-    <inertia ixx="8e-06" ixy="0.0" ixz="-0.0" iyy="4e-06" iyz="-0.0" izz="4e-06"/>
-  </inertial>
-  <visual>
-    <origin rpy="0 0 0" xyz="-0.0659 0.032207 -0.021406"/>
-    <geometry>
-      <mesh filename="package://bot_description/meshes/wheel_right_1.stl" scale="0.001 0.001 0.001"/>
-    </geometry>
-    <material name="silver"/>
-  </visual>
-  <collision>
-    <origin rpy="0 0 0" xyz="-0.0659 0.032207 -0.021406"/>
-    <geometry>
-      <mesh filename="package://bot_description/meshes/wheel_right_1.stl" scale="0.001 0.001 0.001"/>
-    </geometry>
-  </collision>
-</link>
-<link name="wheel_left_1">
-  <inertial>
-    <origin rpy="0 0 0" xyz="0.0033353413496784445 -6.080566113814134e-07 -1.5123052405849324e-07"/>
-    <mass value="0.03301117951419933"/>
-    <inertia ixx="8e-06" ixy="0.0" ixz="0.0" iyy="4e-06" iyz="0.0" izz="4e-06"/>
-  </inertial>
-  <visual>
-    <origin rpy="0 0 0" xyz="0.065896 0.032194 -0.021406"/>
-    <geometry>
-      <mesh filename="package://bot_description/meshes/wheel_left_1.stl" scale="0.001 0.001 0.001"/>
-    </geometry>
-    <material name="silver"/>
-  </visual>
-  <collision>
-    <origin rpy="0 0 0" xyz="0.065896 0.032194 -0.021406"/>
-    <geometry>
-      <mesh filename="package://bot_description/meshes/wheel_left_1.stl" scale="0.001 0.001 0.001"/>
-    </geometry>
-  </collision>
-</link>
-<joint name="Rev3" type="continuous">
-  <origin rpy="0 0 0" xyz="0.021523 0.007087 0.04083"/>
-  <parent link="base_link"/>
-  <child link="rod_1"/>
-  <axis xyz="-0.0 0.0 1.0"/>
-</joint>
-<joint name="Rev4" type="continuous">
-  <origin rpy="0 0 0" xyz="0.0659 -0.032207 0.021406"/>
-  <parent link="base_link"/>
-  <child link="wheel_right_1"/>
-  <axis xyz="-1.0 0.0 -0.0"/>
-</joint>
-<joint name="Rev5" type="continuous">
-  <origin rpy="0 0 0" xyz="-0.065896 -0.032194 0.021406"/>
-  <parent link="base_link"/>
-  <child link="wheel_left_1"/>
-  <axis xyz="1.0 -0.0 0.0"/>
-</joint>
+  <xacro:include filename="$(find bot_description)/urdf/materials_bot.xacro" />
+  <xacro:include filename="$(find bot_description)/urdf/bot_grid.trans" />
+  <xacro:include filename="$(find bot_description)/urdf/bot_grid.gazebo" />
+  <xacro:arg name="bot_uid" default="B1"/>
+  <xacro:macro name="bot_grid_uid" params="uid">
+    <link name="${uid}_base_link">
+      <inertial>
+        <origin rpy="0 0 0" xyz="0.0 0.0 0.027415539003148855"/>
+        <mass value="1.1517833070915058"/>
+        <inertia ixx="0.001068" ixy="-2.4e-05" ixz="-8e-06" iyy="0.000918" iyz="4.8e-05" izz="0.001472"/>
+      </inertial>
+      <visual>
+        <origin rpy="0 0 0" xyz="0 0 0"/>
+        <geometry>
+          <mesh filename="package://bot_description/meshes/base_link.stl" scale="0.001 0.001 0.001"/>
+        </geometry>
+        <material name="silver"/>
+      </visual>
+      <collision>
+        <origin rpy="0 0 0" xyz="0 0 0"/>
+        <geometry>
+          <mesh filename="package://bot_description/meshes/base_link.stl" scale="0.001 0.001 0.001"/>
+        </geometry>
+      </collision>
+    </link>
+    <link name="${uid}_release_rod">
+      <inertial>
+        <origin rpy="0 0 0" xyz="-0.03412970107262531 3.283082382239677e-07 0.000999532672142013"/>
+        <mass value="0.004917856385932786"/>
+        <inertia ixx="0.0" ixy="0.0" ixz="-0.0" iyy="2e-06" iyz="-0.0" izz="2e-06"/>
+      </inertial>
+      <visual>
+        <origin rpy="0 0 0" xyz="-0.021523 -0.007087 -0.04083"/>
+        <geometry>
+          <mesh filename="package://bot_description/meshes/rod_1.stl" scale="0.001 0.001 0.001"/>
+        </geometry>
+        <material name="silver"/>
+      </visual>
+      <collision>
+        <origin rpy="0 0 0" xyz="-0.021523 -0.007087 -0.04083"/>
+        <geometry>
+          <mesh filename="package://bot_description/meshes/rod_1.stl" scale="0.001 0.001 0.001"/>
+        </geometry>
+      </collision>
+    </link>
+    <link name="${uid}_right_wheel">
+      <inertial>
+        <origin rpy="0 0 0" xyz="-0.0033351165545466577 4.777016239451704e-07 -1.512305142191417e-07"/>
+        <mass value="0.03301117951310708"/>
+        <inertia ixx="8e-06" ixy="0.0" ixz="-0.0" iyy="4e-06" iyz="-0.0" izz="4e-06"/>
+      </inertial>
+      <visual>
+        <origin rpy="0 0 0" xyz="-0.0659 0.032207 -0.021406"/>
+        <geometry>
+          <mesh filename="package://bot_description/meshes/wheel_right_1.stl" scale="0.001 0.001 0.001"/>
+        </geometry>
+        <material name="silver"/>
+      </visual>
+      <collision>
+        <origin rpy="0 0 0" xyz="-0.0659 0.032207 -0.021406"/>
+        <geometry>
+          <mesh filename="package://bot_description/meshes/wheel_right_1.stl" scale="0.001 0.001 0.001"/>
+        </geometry>
+      </collision>
+    </link>
+    <link name="${uid}_left_wheel">
+      <inertial>
+        <origin rpy="0 0 0" xyz="0.0033353413496784445 -6.080566113814134e-07 -1.5123052405849324e-07"/>
+        <mass value="0.03301117951419933"/>
+        <inertia ixx="8e-06" ixy="0.0" ixz="0.0" iyy="4e-06" iyz="0.0" izz="4e-06"/>
+      </inertial>
+      <visual>
+        <origin rpy="0 0 0" xyz="0.065896 0.032194 -0.021406"/>
+        <geometry>
+          <mesh filename="package://bot_description/meshes/wheel_left_1.stl" scale="0.001 0.001 0.001"/>
+        </geometry>
+        <material name="silver"/>
+      </visual>
+      <collision>
+        <origin rpy="0 0 0" xyz="0.065896 0.032194 -0.021406"/>
+        <geometry>
+          <mesh filename="package://bot_description/meshes/wheel_left_1.stl" scale="0.001 0.001 0.001"/>
+        </geometry>
+      </collision>
+    </link>
+    <joint name="${uid}_release_servo_joint" type="continuous">
+      <origin rpy="0 0 0" xyz="0.021523 0.007087 0.04083"/>
+      <parent link="${uid}_base_link"/>
+      <child link="${uid}_release_rod"/>
+      <axis xyz="-0.0 0.0 1.0"/>
+    </joint>
+    <joint name="${uid}_right_motor_joint" type="continuous">
+      <origin rpy="0 0 0" xyz="0.0659 -0.032207 0.021406"/>
+      <parent link="${uid}_base_link"/>
+      <child link="${uid}_right_wheel"/>
+      <axis xyz="-1.0 0.0 -0.0"/>
+    </joint>
+    <joint name="${uid}_left_motor_joint" type="continuous">
+      <origin rpy="0 0 0" xyz="-0.065896 -0.032194 0.021406"/>
+      <parent link="${uid}_base_link"/>
+      <child link="${uid}_left_wheel"/>
+      <axis xyz="1.0 -0.0 0.0"/>
+    </joint>
+  </xacro:macro>
+  <xacro:bot_grid_uid uid="$(arg bot_uid)" />
+  <xacro:bot_trans_uid uid="$(arg bot_uid)" />
+  <xacro:bot_gazebo_uid uid="$(arg bot_uid)" />
 </robot>

Commit message: added controller

File: src/bot_description/urdf/bot_grid.xacro (robot description, xacro)
@@ -104,4 +104,40 @@
       <axis xyz="1.0 -0.0 0.0"/>
     </joint>
+    <transmission name="tran1">
+      <type>transmission_interface/SimpleTransmission</type>
+      <joint name="${uid}_release_servo_joint">
+        <hardwareInterface>hardware_interface/EffortJointInterface</hardwareInterface>
+      </joint>
+      <actuator name="servo1">
+        <hardwareInterface>hardware_interface/EffortJointInterface</hardwareInterface>
+        <mechanicalReduction>1</mechanicalReduction>
+      </actuator>
+    </transmission>
+    <transmission name="tran2">
+      <type>transmission_interface/SimpleTransmission</type>
+      <joint name="${uid}_right_motor_joint">
+        <hardwareInterface>hardware_interface/VelocityJointInterface</hardwareInterface>
+      </joint>
+      <actuator name="right_motor">
+        <hardwareInterface>hardware_interface/VelocityJointInterface</hardwareInterface>
+        <mechanicalReduction>1</mechanicalReduction>
+      </actuator>
+    </transmission>
+    <transmission name="tran3">
+      <type>transmission_interface/SimpleTransmission</type>
+      <joint name="${uid}_left_motor_joint">
+        <hardwareInterface>hardware_interface/VelocityJointInterface</hardwareInterface>
+      </joint>
+      <actuator name="left_motor">
+        <hardwareInterface>hardware_interface/VelocityJointInterface</hardwareInterface>
+        <mechanicalReduction>1</mechanicalReduction>
+      </actuator>
+    </transmission>
+    <gazebo>
+      <plugin name="gazebo_ros_control" filename="libgazebo_ros_control.so">
+        <robotNamespace>/bot_grid_controller</robotNamespace>
+        <robotSimType>gazebo_ros_control/DefaultRobotHWSim</robotSimType>
+      </plugin>
+    </gazebo>
   </xacro:macro>
   <xacro:bot_grid_uid uid="$(arg bot_uid)" />

Commit message: Added the mpc package

File: src/bot_description/urdf/bot_grid.xacro (robot description, xacro)
@@ -4,7 +4,5 @@
   <xacro:include filename="$(find bot_description)/urdf/bot_grid.trans" />
   <xacro:include filename="$(find bot_description)/urdf/bot_grid.gazebo" />
-  <xacro:arg name="bot_uid" default="B1"/>
-  <xacro:macro name="bot_grid_uid" params="uid">
-    <link name="${uid}_base_link">
+    <link name="base_body">
       <inertial>
         <origin rpy="0 0 0" xyz="0.0 0.0 0.027415539003148855"/>
@@ -26,5 +24,7 @@
       </collision>
     </link>
-    <link name="${uid}_release_rod">
+    <link name="base_link">
+    </link>
+    <link name="release_rod">
       <inertial>
         <origin rpy="0 0 0" xyz="-0.03412970107262531 3.283082382239677e-07 0.000999532672142013"/>
@@ -46,5 +46,5 @@
       </collision>
     </link>
-    <link name="${uid}_right_wheel">
+    <link name="right_wheel">
       <inertial>
         <origin rpy="0 0 0" xyz="-0.0033351165545466577 4.777016239451704e-07 -1.512305142191417e-07"/>
@@ -66,5 +66,5 @@
       </collision>
     </link>
-    <link name="${uid}_left_wheel">
+    <link name="left_wheel">
       <inertial>
         <origin rpy="0 0 0" xyz="0.0033353413496784445 -6.080566113814134e-07 -1.5123052405849324e-07"/>
@@ -86,25 +86,31 @@
       </collision>
     </link>
-    <joint name="${uid}_release_servo_joint" type="continuous">
+    <joint name="release_servo_joint" type="continuous">
       <origin rpy="0 0 0" xyz="0.021523 0.007087 0.04083"/>
-      <parent link="${uid}_base_link"/>
-      <child link="${uid}_release_rod"/>
+      <parent link="base_link"/>
+      <child link="release_rod"/>
       <axis xyz="-0.0 0.0 1.0"/>
     </joint>
-    <joint name="${uid}_right_motor_joint" type="continuous">
+    <joint name="right_motor_joint" type="continuous">
       <origin rpy="0 0 0" xyz="0.0659 -0.032207 0.021406"/>
-      <parent link="${uid}_base_link"/>
-      <child link="${uid}_right_wheel"/>
+      <parent link="base_link"/>
+      <child link="right_wheel"/>
       <axis xyz="-1.0 0.0 -0.0"/>
     </joint>
-    <joint name="${uid}_left_motor_joint" type="continuous">
+    <joint name="left_motor_joint" type="continuous">
       <origin rpy="0 0 0" xyz="-0.065896 -0.032194 0.021406"/>
-      <parent link="${uid}_base_link"/>
-      <child link="${uid}_left_wheel"/>
+      <parent link="base_link"/>
+      <child link="left_wheel"/>
       <axis xyz="1.0 -0.0 0.0"/>
+    </joint>
+    <joint name="base_joint" type="fixed">
+      <origin rpy="0.0 0.0 0.0" xyz="0.0 0.0 0.0"/>
+      <parent link="base_link"/>
+      <child link="base_body"/>
+      <axis xyz="0.0 0.0 0.0"/>
     </joint>
     <transmission name="tran1">
       <type>transmission_interface/SimpleTransmission</type>
-      <joint name="${uid}_release_servo_joint">
+      <joint name="release_servo_joint">
         <hardwareInterface>hardware_interface/EffortJointInterface</hardwareInterface>
       </joint>
@@ -116,5 +122,5 @@
     <transmission name="tran2">
       <type>transmission_interface/SimpleTransmission</type>
-      <joint name="${uid}_right_motor_joint">
+      <joint name="right_motor_joint">
         <hardwareInterface>hardware_interface/VelocityJointInterface</hardwareInterface>
       </joint>
@@ -126,5 +132,5 @@
     <transmission name="tran3">
       <type>transmission_interface/SimpleTransmission</type>
-      <joint name="${uid}_left_motor_joint">
+      <joint name="left_motor_joint">
         <hardwareInterface>hardware_interface/VelocityJointInterface</hardwareInterface>
       </joint>
@@ -140,7 +146,3 @@
       </plugin>
     </gazebo>
-  </xacro:macro>
-  <xacro:bot_grid_uid uid="$(arg bot_uid)" />
-  <xacro:bot_trans_uid uid="$(arg bot_uid)" />
-  <xacro:bot_gazebo_uid uid="$(arg bot_uid)" />
 </robot>
